Commit message: Single leg digital twin completed

File: urdf/robot_backup.urdf (robot description, URDF)
Before this commit: robot 09.06.26_5pm, 12 links, 11 joints
Links:
- link actuator_1_v1_1: geometry collision mesh filename=../meshes/actuator_1_v1_1.stl scale=0.001 0.001 0.001; visual mesh filename=../meshes/actuator_1_v1_1.stl scale=0.001 0.001 0.001
- link actuator_2_v1_1: geometry collision mesh filename=../meshes/actuator_2_v1_1.stl scale=0.001 0.001 0.001; visual mesh filename=../meshes/actuator_2_v1_1.stl scale=0.001 0.001 0.001
- link ankle_bearing_v1_1: geometry collision mesh filename=../meshes/ankle_bearing_v1_1.stl scale=0.001 0.001 0.001; visual mesh filename=../meshes/ankle_bearing_v1_1.stl scale=0.001 0.001 0.001
- link ankle_bracelet_v1_1: geometry collision mesh filename=../meshes/ankle_bracelet_v1_1.stl scale=0.001 0.001 0.001; visual mesh filename=../meshes/ankle_bracelet_v1_1.stl scale=0.001 0.001 0.001
- link ankle_clevis_v1_1: geometry collision mesh filename=../meshes/ankle_clevis_v1_1.stl scale=0.001 0.001 0.001; visual mesh filename=../meshes/ankle_clevis_v1_1.stl scale=0.001 0.001 0.001
- link base_link: geometry collision mesh filename=../meshes/base_link.stl scale=0.001 0.001 0.001; visual mesh filename=../meshes/base_link.stl scale=0.001 0.001 0.001
- link hip_clevis_v1_1: geometry collision mesh filename=../meshes/hip_clevis_v1_1.stl scale=0.001 0.001 0.001; visual mesh filename=../meshes/hip_clevis_v1_1.stl scale=0.001 0.001 0.001
- link knee_bearing_holder_v1_1: geometry collision mesh filename=../meshes/knee_bearing_holder_v1_1.stl scale=0.001 0.001 0.001; visual mesh filename=../meshes/knee_bearing_holder_v1_1.stl scale=0.001 0.001 0.001
- link knee_bearing_v1_1: geometry collision mesh filename=../meshes/knee_bearing_v1_1.stl scale=0.001 0.001 0.001; visual mesh filename=../meshes/knee_bearing_v1_1.stl scale=0.001 0.001 0.001
- link leg_1_rod_v1_1: geometry collision mesh filename=../meshes/leg_1_rod_v1_1.stl scale=0.001 0.001 0.001; visual mesh filename=../meshes/leg_1_rod_v1_1.stl scale=0.001 0.001 0.001
- link leg_2_rod_v1_1: geometry collision mesh filename=../meshes/leg_2_rod_v1_1.stl scale=0.001 0.001 0.001; visual mesh filename=../meshes/leg_2_rod_v1_1.stl scale=0.001 0.001 0.001
- link leg_stack_v1_1: geometry collision mesh filename=../meshes/leg_stack_v1_1.stl scale=0.001 0.001 0.001; visual mesh filename=../meshes/leg_stack_v1_1.stl scale=0.001 0.001 0.001
